File: GPIOLabel.kicad_pcb (KiCad board)
At the start: 2 copper layers, 20.3 x 66 mm, 2 parts, among them M1 MountingHole_3.2mm_M3_DIN965_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, P1 CONN_02X20

Commit message: rename ios with just numbers, center, cleanup
Other:
- board size 20.3 x 66 mm -> 20.3 x 67 mm
- board text added: "10"
- board text added: "11"
- board text added: "12"
- board text added: "13"
- board text added: "14"
- board text added: "15"
- board text added: "16"
- board text added: "17"
- board text added: "18"
- board text added: "19"
- board text added: "20"
- board text added: "21"
- board text added: "22"
- board text added: "23"
- board text added: "24"
- board text added: "25"
- board text added: "26"
- board text added: "27"
- board text added: "3"
- board text added: "4"
- board text added: "5"
- board text added: "6"
- board text added: "7"
- board text added: "8"
- board text added: "9"
- board text added: "ID_SC"
- board text added: "ID_SD"
- board text removed: "1"
- board text removed: "GPIO0"
- board text removed: "GPIO1"
- board text removed: "GPIO10"
- board text removed: "GPIO11"
- board text removed: "GPIO12"
- board text removed: "GPIO13"
- board text removed: "GPIO14"
- board text removed: "GPIO15"
- board text removed: "GPIO16"
- board text removed: "GPIO17"
- board text removed: "GPIO18"
- board text removed: "GPIO19"
- board text removed: "GPIO2"
- board text removed: "GPIO20"
- board text removed: "GPIO21"
- board text removed: "GPIO22"
- board text removed: "GPIO23"
- board text removed: "GPIO24"
- board text removed: "GPIO25"
- board text removed: "GPIO26"
- board text removed: "GPIO27"
- board text removed: "GPIO3"
- board text removed: "GPIO4"
- board text removed: "GPIO5"
- board text removed: "GPIO6"
- board text removed: "GPIO7"
- board text removed: "GPIO8"
- board text removed: "GPIO9"
